File: POC/PCB/LedCC_Side/LedCC_Side.kicad_pcb (KiCad board)
At the start: 2 copper layers, 84.5 x 19.7 mm, 19 parts, among them J1 In, J2 Out, J3 In, J4 Out

Commit message: Testing code updates
Other:
- board text added: "V"
