File: PCB/LedCC_Side/LedCC_Side.kicad_sch (KiCad schematic)
At the start: 19 parts, among them J1 In, J2 Out, J3 In, J4 Out

Commit message: PCB Updates
Parts:
- removed H1, H2: MountingHole, MountingHole:MountingHole_2.2mm_M2, symbol Mechanical:MountingHole
- removed J1, J3: In, Library:Led-Jumper, symbol Connector_Generic:Conn_01x03
- removed J2, J4: Out, Library:Led-Jumper, symbol Connector_Generic:Conn_01x03
- removed R1: 330, Resistor_SMD:R_0603_1608Metric, symbol Device:R_Small
- added J1, J2, J3, J4, J5, J6: Conn_01x04, Library:HDR-SMD_4P-P1.27-V-M-R2-C2-S1.27-LS5.5, symbol Library:Conn_01x04
- added JP2, JP3, JP4, JP5, JP6: Jumper_2_Small_Bridged, Jumper:SolderJumper-2_P1.3mm_Bridged_RoundedPad1.0x1.5mm, symbol Jumper:Jumper_2_Small_Bridged
Connections:
- net GND: now also J1.3 (Pin_3), J2.3 (Pin_3), J3.3 (Pin_3), J4.3 (Pin_3), J5.3 (Pin_3), J6.3 (Pin_3)
- net VDD: now also J1.4 (Pin_4), J2.4 (Pin_4), J3.4 (Pin_4), J4.4 (Pin_4), J5.4 (Pin_4), J6.4 (Pin_4)
- net at L6.1 (DIN): now also J6.1 (Pin_1), JP6.2 (B); no longer L5.3 (DOUT)
- net at L5.1 (DIN): now also J5.1 (Pin_1), JP5.2 (B); no longer L4.3 (DOUT)
- net Din: now reaches L1.1 (DIN)
- net Din: now also J1.1 (Pin_1)
- net at L2.1 (DIN): now also J2.1 (Pin_1), JP2.2 (B); no longer L1.3 (DOUT)
- net at L2.3 (DOUT): now also J2.2 (Pin_2), JP3.1 (A); no longer L3.1 (DIN)
- net at L4.1 (DIN): now also J4.1 (Pin_1), JP4.2 (B); no longer L3.3 (DOUT)
- net DOUT: no longer names the net of L6.3 (DOUT)
- net DOUT: now also J6.2 (Pin_2)
- new net: J5.2 (Pin_2), JP6.1 (A), L5.3 (DOUT)
- new net: J4.2 (Pin_2), JP5.1 (A), L4.3 (DOUT)
- new net: J3.1 (Pin_1), JP3.2 (B), L3.1 (DIN)
- new net: J3.2 (Pin_2), JP4.1 (A), L3.3 (DOUT)
- new net Dout: J1.2 (Pin_2), JP2.1 (A), L1.3 (DOUT)
Other:
- moved on the sheet: C1, C2, C3, C4, C5, C6, L1, L2, L3, L4, L5, L6
